File: punch-replica/punch-replica.kicad_sch (KiCad schematic)
At the start: 66 parts, among them J1 12V PSU, J10 Screw_Terminal_01x03, J11 Screw_Terminal_01x02, J2 5V OUT, J3 3V3 OUT, J4 LOAD CELL, J5 COIN SLOT, J6 Conn_01x02_Socket, J7 Conn_01x02_Socket, J8 IDC_Connector, J9 Screw_Terminal_01x03, K1 SRD-05VDC-SL-C, K2 SRD-05VDC-SL-C, Q1 BSS138, Q2 BSS138, Q3 Q_NMOS_Depletion_GSD, Q4 Q_NMOS_Depletion_GSD, SW1 SW_Push, SW2 SW_Push, U1 LM2596S-5, U2 AMS1117-3.3, U3 CH340C, U4 PC817, U5 PC817, U6 ESP32-WROOM-32, U7 DFR0299

Commit message: pcb parts placement
Parts:
- removed J3: 3V3 OUT, TerminalBlock:TerminalBlock_MaiXu_MX126-5.0-02P_1x02_P5.00mm, symbol Connector:Screw_Terminal_01x02
- removed J7: Conn_01x02_Socket, Connector_JST:JST_EH_B2B-EH-A_1x02_P2.50mm_Vertical, symbol Connector:Conn_01x02_Socket
- added J4: 5V OUT, TerminalBlock:TerminalBlock_MaiXu_MX126-5.0-02P_1x02_P5.00mm, symbol Connector:Screw_Terminal_01x02
- renumbered J9 to J10, J10 to J11, J11 to J12, J1 to J2, J2 to J3, J4 to J5, J5 to J6, J6 to J7, J8 to J9
Connections:
- net +5V: now also J4.1 (Pin_1)
- net GND: now also J4.2 (Pin_2)
- net P10_LAT: now reaches U6.24 (IO2)
- net P10_LAT: now also J9.10 (Pin_10)
- net P10_DR: now reaches U6.37 (IO23)
- net P10_DR: now also J9.12 (Pin_12)
- net IO13: no longer names the net of U6.16 (IO13)
- net IO13: no longer J9.4 (Pin_4)
- net IO14: no longer names the net of U6.13 (IO14)
- net IO14: no longer J9.2 (Pin_2)
- net IO18 renamed P10_CLK
- net IO19 renamed P10_A
- net P10_A: now also J9.2 (Pin_2); no longer J9.10 (Pin_10)
- net IO21 renamed P10_B
- net P10_B: now also J9.4 (Pin_4); no longer J9.12 (Pin_12)
- net IO22 renamed P10_OE
Other:
- moved on the sheet: J9

Commit message: -
Connections:
- net +5V: now also J5.2 (Pin_2); no longer J5.4 (Pin_4)
- net ESP_ADC1: now also J5.4 (Pin_4); no longer J5.2 (Pin_2)
- net ESP_ADC2: now also J5.5 (Pin_5); no longer J5.3 (Pin_3)
- net GND: now also J5.3 (Pin_3); no longer J5.5 (Pin_5)

Commit message: - adjustment
Parts:
- removed J7: Conn_01x02_Socket, Connector_PinHeader_2.54mm:PinHeader_1x02_P2.54mm_Vertical, symbol Connector:Conn_01x02_Socket
- added C21, C25: 10uF, Capacitor_SMD:C_0805_2012Metric_Pad1.18x1.45mm_HandSolder, symbol Device:C
- added C23, C26: 100uF, Capacitor_SMD:C_1210_3225Metric_Pad1.33x2.70mm_HandSolder, symbol Device:C_Polarized
- added D10: LED, LED_SMD:LED_0805_2012Metric_Pad1.15x1.40mm_HandSolder, symbol Device:LED
- added D11: 1N4001, Diode_SMD:D_SOD-123F, symbol pspice:DIODE
- added J1: Screw_Terminal_01x03, TerminalBlock_Phoenix:TerminalBlock_Phoenix_MKDS-1,5-3_1x03_P5.00mm_Horizontal, symbol Connector:Screw_Terminal_01x03
- added K3: SRD-05VDC-SL-C, Relay_THT:Relay_SPDT_SANYOU_SRD_Series_Form_C, symbol Relay:SANYOU_SRD_Form_C
- added Q5: Q_NMOS_Depletion_GSD, Package_TO_SOT_SMD:SOT-23-3, symbol Device:Q_NMOS_Depletion_GSD
- added R15: 470, Resistor_SMD:R_0603_1608Metric_Pad0.98x0.95mm_HandSolder, symbol Device:R
- added R16: 1k, Resistor_SMD:R_0603_1608Metric_Pad0.98x0.95mm_HandSolder, symbol Device:R
- added R17: 10K, Resistor_SMD:R_0603_1608Metric_Pad0.98x0.95mm_HandSolder, symbol Device:R
- added U28: B0505S-2WR3, Library:B_S-2WR2_MNS, symbol 2024-08-29_08-56-51:B0505S-2WR3
- added U8: PC817, Library:APC-817xx-SL_AMB, symbol Isolator:PC817
- L1: footprint Inductor_SMD:L_Chilisin_BMRF00101040 -> 470; LCSC C408490 -> C475918
Connections:
- net +5V: now also U1.4 (FB), C21.2, C23.1, U28.1 (VIN), U8.1; no longer D7.2 (A), D8.2 (A), K1.5, K2.5, R10.1, R9.1, U4.4, U5.4
- net GND: now also C21.1, C23.2, U28.2 (GND)
- net GNDPWR: now also C25.1, C26.2, Q5.2 (S), R17.2, U28.4 (0V)
- net DC_DRV_3: now reaches U6.8 (IO32)
- net DC_DRV_3: now also R15.1
- new net: D10.1 (K), D11.1 (K), K3.2, Q5.3 (D)
- new net: D10.2 (A), R16.2
- new net: R15.2, U8.2
- new net: Q5.1 (G), R17.1, U8.3
- new net +5VA: C25.2, C26.1, D11.2 (A), D7.2 (A), D8.2 (A), K1.5, K2.5, K3.5, R10.1, R16.1, R9.1, U28.6 (+VO), U4.4, U5.4, U8.4
- new net COM3: J1.2 (Pin_2), K3.1
- new net NC3: J1.1 (Pin_1), K3.4
- new net NO3: J1.3 (Pin_3), K3.3
- no-connect marks 37 -> 36
Other:
- note added: "Output Capacity 5V, 400mA"
- moved on the sheet: D7, D8, J10, J11, K1, K2, Q3, Q4, R10, R11, R12, R6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
